Commit message: Update URDF visual meshes.

File: abb_irb1200_support/urdf/irb1200_7_70_macro.xacro (robot description, xacro)
@@ -14,5 +14,6 @@
       <visual name="visual">
         <geometry>
-          <mesh filename="package://abb_irb1200_support/meshes/irb1200_7_70/visual/base_link.stl" />
+	        <!-- reference irb1200_5_90 package since mesh is shared-->
+          <mesh filename="package://abb_irb1200_support/meshes/irb1200_5_90/visual/base_link.dae" scale="0.001 0.001 0.001" />
         </geometry>
         <material name="graphite_white">
@@ -30,5 +31,6 @@
       <visual name="visual">
         <geometry>
-          <mesh filename="package://abb_irb1200_support/meshes/irb1200_7_70/visual/link_1.stl" />
+	        <!-- reference irb1200_5_90 package since mesh is shared-->
+          <mesh filename="package://abb_irb1200_support/meshes/irb1200_5_90/visual/link_1.dae" scale="0.001 0.001 0.001" />
         </geometry>
         <material name="graphite_white"/>
@@ -44,5 +46,5 @@
       <visual name="visual">
         <geometry>
-          <mesh filename="package://abb_irb1200_support/meshes/irb1200_7_70/visual/link_2.stl" />
+          <mesh filename="package://abb_irb1200_support/meshes/irb1200_7_70/visual/link_2.dae" scale="0.001 0.001 0.001" />
         </geometry>
         <material name="graphite_white"/>
@@ -58,5 +60,5 @@
       <visual name="visual">
         <geometry>
-          <mesh filename="package://abb_irb1200_support/meshes/irb1200_7_70/visual/link_3.stl" />
+          <mesh filename="package://abb_irb1200_support/meshes/irb1200_7_70/visual/link_3.dae" scale="0.001 0.001 0.001" />
         </geometry>
         <material name="graphite_white"/>
@@ -72,5 +74,6 @@
       <visual name="visual">
         <geometry>
-          <mesh filename="package://abb_irb1200_support/meshes/irb1200_7_70/visual/link_4.stl" />
+	        <!-- reference irb1200_5_90 package since mesh is shared-->
+          <mesh filename="package://abb_irb1200_support/meshes/irb1200_5_90/visual/link_4.dae" scale="0.001 0.001 0.001" />
         </geometry>
         <material name="graphite_white"/>
@@ -86,5 +89,6 @@
       <visual name="visual">
         <geometry>
-          <mesh filename="package://abb_irb1200_support/meshes/irb1200_7_70/visual/link_5.stl" />
+	        <!-- reference irb1200_5_90 package since mesh is shared-->
+          <mesh filename="package://abb_irb1200_support/meshes/irb1200_5_90/visual/link_5.dae" scale="0.001 0.001 0.001" />
         </geometry>
         <material name="graphite_white"/>
@@ -100,5 +104,6 @@
       <visual name="visual">
         <geometry>
-          <mesh filename="package://abb_irb1200_support/meshes/irb1200_7_70/visual/link_6.stl" />
+	        <!-- reference irb1200_5_90 package since mesh is shared-->
+          <mesh filename="package://abb_irb1200_support/meshes/irb1200_5_90/visual/link_6.dae" scale="0.001 0.001 0.001" />
         </geometry>
         <material name="graphite_white"/>

Commit message: Update 7_70 mesh origins

File: abb_irb1200_support/urdf/irb1200_7_70_macro.xacro (robot description, xacro)
@@ -15,5 +15,5 @@
         <geometry>
 	        <!-- reference irb1200_5_90 package since mesh is shared-->
-          <mesh filename="package://abb_irb1200_support/meshes/irb1200_5_90/visual/base_link.dae" scale="0.001 0.001 0.001" />
+          <mesh filename="package://abb_irb1200_support/meshes/irb1200_5_90/visual/base_link.dae"  />
         </geometry>
         <material name="graphite_white">
@@ -32,5 +32,5 @@
         <geometry>
 	        <!-- reference irb1200_5_90 package since mesh is shared-->
-          <mesh filename="package://abb_irb1200_support/meshes/irb1200_5_90/visual/link_1.dae" scale="0.001 0.001 0.001" />
+          <mesh filename="package://abb_irb1200_support/meshes/irb1200_5_90/visual/link_1.dae" />
         </geometry>
         <material name="graphite_white"/>
@@ -46,5 +46,5 @@
       <visual name="visual">
         <geometry>
-          <mesh filename="package://abb_irb1200_support/meshes/irb1200_7_70/visual/link_2.dae" scale="0.001 0.001 0.001" />
+          <mesh filename="package://abb_irb1200_support/meshes/irb1200_7_70/visual/link_2.dae" />
         </geometry>
         <material name="graphite_white"/>
@@ -60,5 +60,5 @@
       <visual name="visual">
         <geometry>
-          <mesh filename="package://abb_irb1200_support/meshes/irb1200_7_70/visual/link_3.dae" scale="0.001 0.001 0.001" />
+          <mesh filename="package://abb_irb1200_support/meshes/irb1200_7_70/visual/link_3.dae" />
         </geometry>
         <material name="graphite_white"/>
@@ -75,5 +75,5 @@
         <geometry>
 	        <!-- reference irb1200_5_90 package since mesh is shared-->
-          <mesh filename="package://abb_irb1200_support/meshes/irb1200_5_90/visual/link_4.dae" scale="0.001 0.001 0.001" />
+          <mesh filename="package://abb_irb1200_support/meshes/irb1200_7_70/visual/link_4.dae" />
         </geometry>
         <material name="graphite_white"/>
@@ -90,5 +90,5 @@
         <geometry>
 	        <!-- reference irb1200_5_90 package since mesh is shared-->
-          <mesh filename="package://abb_irb1200_support/meshes/irb1200_5_90/visual/link_5.dae" scale="0.001 0.001 0.001" />
+          <mesh filename="package://abb_irb1200_support/meshes/irb1200_5_90/visual/link_5.dae" />
         </geometry>
         <material name="graphite_white"/>
@@ -105,5 +105,5 @@
         <geometry>
 	        <!-- reference irb1200_5_90 package since mesh is shared-->
-          <mesh filename="package://abb_irb1200_support/meshes/irb1200_5_90/visual/link_6.dae" scale="0.001 0.001 0.001" />
+          <mesh filename="package://abb_irb1200_support/meshes/irb1200_5_90/visual/link_6.dae" />
         </geometry>
         <material name="graphite_white"/>
