Commit message: Change joint limits to match our robot
This is a hack until we update trac_ik to use moveit's new IK interface,
which will let us pass joint limits to the IK solver from params.

File: abb_irb1200_support/urdf/irb1200_5_90_macro.xacro (robot description, xacro)
@@ -153,5 +153,7 @@
       <parent link="${prefix}link_2"/>
       <child link="${prefix}link_3"/>
-      <limit effort="0" lower="-3.491" upper="1.222" velocity="5.236"/>
+      <!-- Original values: <limit effort="0" lower="-3.491" upper="1.222" velocity="5.236"/> -->
+      <!-- Hacked limits for our robot since trac_ik doesn't yet get joint limits from params: -->
+      <limit effort="0" lower="-0.5" upper="1.2" velocity="5.236"/>
     </joint>
     <joint type="revolute" name="${prefix}joint_4">
@@ -160,5 +162,7 @@
       <parent link="${prefix}link_3"/>
       <child link="${prefix}link_4"/>
-      <limit effort="0" lower="-4.712" upper="4.712" velocity="6.981"/>
+      <!-- Original values: <limit effort="0" lower="-4.712" upper="4.712" velocity="6.981"/> -->
+      <!-- Hacked limits for our robot since trac_ik doesn't yet get joint limits from params: -->
+       <limit effort="0" lower="-2.8" upper="2.8" velocity="6.981"/>
     </joint>
     <joint type="revolute" name="${prefix}joint_5">

Commit message: Calculate inertial using meshlab
All inertials blocks were calculated with meshlab + some basic octave
script except for link6. When using the calculated values the robot
"crashed" when rotating it.

File: abb_irb1200_support/urdf/irb1200_5_90_macro.xacro (robot description, xacro)
@@ -5,7 +5,7 @@
     <link name="${prefix}base_link">
       <inertial>
-        <mass value="6.215"/>
-        <origin xyz="-0.04204 8.01E-05 0.07964" rpy="0 0 0"/>
-        <inertia ixx="0.0247272" ixy="-8.0784E-05" ixz="0.00130902" iyy="0.0491285" iyz="-8.0419E-06" izz="0.0472376"/>
+        <mass value="13.7742"/>
+        <origin xyz="-0.028986 0.000596 0.11273"/>
+        <inertia ixx="0.101998" ixy="0.000495482" ixz="0.000311158" iyy="0.13969" iyz="-0.000245375" izz="0.130433"/>
       </inertial>
       <collision name="collision">
@@ -25,7 +25,7 @@
     <link name="${prefix}link_1">
       <inertial>
-        <mass value="3.067" />
-        <origin xyz="9.77E-05 -0.00012 0.23841" rpy="0 0 0"/>
-        <inertia ixx="0.0142175" ixy="-1.28579E-05" ixz="-2.31364E-05" iyy="0.0144041" iyz="1.93404E-05" izz="0.0104533"/>
+        <mass value="11.8419"/>
+        <origin xyz="0.000877 -0.000631 0.336217"/>
+        <inertia ixx="0.11194" ixy="-4.54988e-05" ixz="0.000280961" iyy="0.0915158" iyz="-0.000109905" izz="0.0876456"/>
       </inertial>
       <collision name="collision">
@@ -43,7 +43,7 @@
     <link name="${prefix}link_2">
       <inertial>
-        <mass value="3.909"/>
-        <origin xyz="0.00078 -0.00212 0.10124" rpy="0 0 0"/>
-        <inertia ixx="0.0603111" ixy="9.83431E-06" ixz="5.72407E-05" iyy="0.041569" iyz="-0.00050497" izz="0.0259548"/>
+        <mass value="17.5394"/>
+        <origin xyz="-0.000928 -0.000497 0.250051"/>
+        <inertia ixx="0.493558" ixy="1.32136e-05" ixz="0.000209024" iyy="0.462939" iyz="-0.00179901" izz="0.0894214"/>
       </inertial>
       <collision name="collision">
@@ -61,7 +61,7 @@
     <link name="${prefix}link_3">
       <inertial>
-        <mass value="2.944"/>
-        <origin xyz="0.02281 0.00106 0.05791" rpy="0 0 0"/>
-        <inertia ixx="0.00835606" ixy="-8.01545E-05" ixz="0.00142884" iyy="0.016713" iyz="-0.000182227" izz="0.0126984"/>
+        <mass value="7.46365"/>
+        <origin xyz="0.099588 0.001143 0.032333"/>
+        <inertia ixx="0.0252424" ixy="0.000142737" ixz="-0.00565542" iyy="0.0906438" iyz="0.000142213" izz="0.0825079"/>
       </inertial>
       <collision name="collision">
@@ -79,7 +79,7 @@
     <link name="${prefix}link_4">
       <inertial>
-        <mass value="1.328"/>
-        <origin xyz="0.2247 0.00015 0.00041" rpy="0 0 0"/>
-        <inertia ixx="0.00284661" ixy="-2.12765E-05" ixz="-1.6435E-05" iyy="0.00401346" iyz="1.31336E-05" izz="0.0052535"/>
+        <mass value="2.74436"/>
+        <origin xyz="0.381678 0.001261 0.005168"/>
+        <inertia ixx="0.00573099" ixy="-0.000131119" ixz="0.000380232" iyy="0.0118352" iyz="-2.26565e-05" izz="0.0114428"/>
       </inertial>
       <collision name="collision">
@@ -97,7 +97,7 @@
     <link name="${prefix}link_5">
       <inertial>
-        <mass value="0.546"/>
-        <origin xyz="-0.00109 3.68E-05 6.22E-05" rpy="0 0 0"/>
-        <inertia ixx="0.000404891" ixy="1.61943E-06" ixz="8.46805E-07" iyy="0.000892825" iyz="-1.51792E-08" izz="0.000815468"/>
+        <mass value="0.62953"/>
+        <origin xyz="0.011197 -0.001056 0.000109"/>
+        <inertia ixx="0.000502815" ixy="-1.03173e-05" ixz="-8.74347e-08" iyy="0.00108856" iyz="2.07657e-07" izz="0.000918873"/>
       </inertial>
       <collision name="collision">
@@ -119,4 +119,12 @@
         <inertia ixx="0.001" ixy="0" ixz="0" iyy="0.001" iyz="0" izz="0.001"/>
       </inertial>
+      <!--
+      Meshlab calculated values make the robot crash when rotating this joint.
+      <inertial>
+        <mass value="0.00686711"/>
+        <origin xyz="-0.00250976 -1.89e-06 0.00010218"/>
+        <inertia ixx="1.3517e-06" ixy="-1.21316e-11" ixz="9.18065e-12" iyy="6.89813e-07" iyz="-1.21534e-10" izz="6.90097e-07"/>
+      </inertial>
+      -->
       <collision name="collision">
         <geometry>

Commit message: Tune joint dynamics + controller PIDs

File: abb_irb1200_support/urdf/irb1200_5_90_macro.xacro (robot description, xacro)
@@ -148,5 +148,5 @@
       <child link="${prefix}link_1"/>
       <limit effort="10000" lower="-2.967" upper="2.967" velocity="5.027"/>
-      <dynamics damping="1.0" friction="1.0"/>
+      <dynamics damping="50.0" friction="1.0"/>
     </joint>
     <joint type="revolute" name="${prefix}joint_2">
@@ -156,5 +156,5 @@
       <child link="${prefix}link_2"/>
       <limit effort="10000" lower="-1.745" upper="2.269" velocity="4.189"/>
-      <dynamics damping="1.0" friction="1.0"/>
+      <dynamics damping="50.0" friction="1.0"/>
     </joint>
     <joint type="revolute" name="${prefix}joint_3">
@@ -166,5 +166,5 @@
       <!-- Hacked limits for our robot since trac_ik doesn't yet get joint limits from params: -->
       <limit effort="10000" lower="-0.5" upper="1.2" velocity="5.236"/>
-      <dynamics damping="1.0" friction="1.0"/>
+      <dynamics damping="10.0" friction="1.0"/>
     </joint>
     <joint type="revolute" name="${prefix}joint_4">
@@ -176,5 +176,5 @@
       <!-- Hacked limits for our robot since trac_ik doesn't yet get joint limits from params: -->
        <limit effort="10000" lower="-2.8" upper="2.8" velocity="6.981"/>
-      <dynamics damping="1.0" friction="1.0"/>
+      <dynamics damping="5.0" friction="1.0"/>
     </joint>
     <joint type="revolute" name="${prefix}joint_5">
@@ -184,5 +184,5 @@
       <child link="${prefix}link_5"/>
       <limit effort="10000" lower="-2.269" upper="2.269" velocity="7.069"/>
-      <dynamics damping="1.0" friction="1.0"/>
+      <dynamics damping="2.0" friction="1.0"/>
     </joint>
     <joint type="revolute" name="${prefix}joint_6">
