Commit message: Effort controllers for irb1200

File: abb_irb1200_gazebo/urdf/irb1200_5_90_macro.xacro (robot description, xacro)
@@ -6,5 +6,5 @@
       <type>transmission_interface/SimpleTransmission</type>
       <joint name="${prefix}joint_1">
-        <hardwareInterface>hardware_interface/PositionJointInterface</hardwareInterface>
+        <hardwareInterface>hardware_interface/EffortJointInterface</hardwareInterface>
       </joint>
       <actuator name="${prefix}motor1">
@@ -15,5 +15,5 @@
       <type>transmission_interface/SimpleTransmission</type>
       <joint name="${prefix}joint_2">
-        <hardwareInterface>hardware_interface/PositionJointInterface</hardwareInterface>
+        <hardwareInterface>hardware_interface/EffortJointInterface</hardwareInterface>
       </joint>
       <actuator name="${prefix}motor2">
@@ -24,5 +24,5 @@
       <type>transmission_interface/SimpleTransmission</type>
       <joint name="${prefix}joint_3">
-        <hardwareInterface>hardware_interface/PositionJointInterface</hardwareInterface>
+        <hardwareInterface>hardware_interface/EffortJointInterface</hardwareInterface>
       </joint>
       <actuator name="${prefix}motor3">
@@ -33,5 +33,5 @@
       <type>transmission_interface/SimpleTransmission</type>
       <joint name="${prefix}joint_4">
-        <hardwareInterface>hardware_interface/PositionJointInterface</hardwareInterface>
+        <hardwareInterface>hardware_interface/EffortJointInterface</hardwareInterface>
       </joint>
       <actuator name="${prefix}motor4">
@@ -42,5 +42,5 @@
       <type>transmission_interface/SimpleTransmission</type>
       <joint name="${prefix}joint_5">
-        <hardwareInterface>hardware_interface/PositionJointInterface</hardwareInterface>
+        <hardwareInterface>hardware_interface/EffortJointInterface</hardwareInterface>
       </joint>
       <actuator name="${prefix}motor5">
@@ -51,5 +51,5 @@
       <type>transmission_interface/SimpleTransmission</type>
       <joint name="${prefix}joint_6">
-        <hardwareInterface>hardware_interface/PositionJointInterface</hardwareInterface>
+        <hardwareInterface>hardware_interface/EffortJointInterface</hardwareInterface>
       </joint>
       <actuator name="${prefix}motor6">

File: abb_irb1200_support/urdf/irb1200_5_90_macro.xacro (robot description, xacro)
@@ -139,5 +139,6 @@
       <parent link="${prefix}base_link"/>
       <child link="${prefix}link_1"/>
-      <limit effort="0" lower="-2.967" upper="2.967" velocity="5.027"/>
+      <limit effort="10000" lower="-2.967" upper="2.967" velocity="5.027"/>
+      <dynamics damping="1.0" friction="1.0"/>
     </joint>
     <joint type="revolute" name="${prefix}joint_2">
@@ -146,5 +147,6 @@
       <parent link="${prefix}link_1"/>
       <child link="${prefix}link_2"/>
-      <limit effort="0" lower="-1.745" upper="2.269" velocity="4.189"/>
+      <limit effort="10000" lower="-1.745" upper="2.269" velocity="4.189"/>
+      <dynamics damping="1.0" friction="1.0"/>
     </joint>
     <joint type="revolute" name="${prefix}joint_3">
@@ -155,5 +157,6 @@
       <!-- Original values: <limit effort="0" lower="-3.491" upper="1.222" velocity="5.236"/> -->
       <!-- Hacked limits for our robot since trac_ik doesn't yet get joint limits from params: -->
-      <limit effort="0" lower="-0.5" upper="1.2" velocity="5.236"/>
+      <limit effort="10000" lower="-0.5" upper="1.2" velocity="5.236"/>
+      <dynamics damping="1.0" friction="1.0"/>
     </joint>
     <joint type="revolute" name="${prefix}joint_4">
@@ -164,5 +167,6 @@
       <!-- Original values: <limit effort="0" lower="-4.712" upper="4.712" velocity="6.981"/> -->
       <!-- Hacked limits for our robot since trac_ik doesn't yet get joint limits from params: -->
-       <limit effort="0" lower="-2.8" upper="2.8" velocity="6.981"/>
+       <limit effort="10000" lower="-2.8" upper="2.8" velocity="6.981"/>
+      <dynamics damping="1.0" friction="1.0"/>
     </joint>
     <joint type="revolute" name="${prefix}joint_5">
@@ -171,5 +175,6 @@
       <parent link="${prefix}link_4"/>
       <child link="${prefix}link_5"/>
-      <limit effort="0" lower="-2.269" upper="2.269" velocity="7.069"/>
+      <limit effort="10000" lower="-2.269" upper="2.269" velocity="7.069"/>
+      <dynamics damping="1.0" friction="1.0"/>
     </joint>
     <joint type="revolute" name="${prefix}joint_6">
@@ -178,5 +183,6 @@
       <parent link="${prefix}link_5"/>
       <child link="${prefix}link_6"/>
-      <limit effort="0" lower="-6.283" upper="6.283" velocity="10.472"/>
+      <limit effort="10000" lower="-6.283" upper="6.283" velocity="10.472"/>
+      <dynamics damping="1.0" friction="1.0"/>
     </joint>
     <joint type="fixed" name="${prefix}joint_6-tool0">
